Commit message: visualized hand

File: franka_description/panda.urdf (robot description, URDF)
Before this commit: robot panda, 17 links, 16 joints
Links:
- added link left_inner_finger, mass 0.00724255346165745; collision mesh filename=robotiq_arg85_description/meshes/inner_finger_coarse.STL; visual mesh filename=robotiq_arg85_description/meshes/inner_finger_fine.STL
- added link left_inner_knuckle, mass 0.0110930853895903; collision mesh filename=robotiq_arg85_description/meshes/inner_knuckle_coarse.STL; visual mesh filename=robotiq_arg85_description/meshes/inner_knuckle_fine.STL
- added link left_outer_finger, mass 0.0273093985570947; collision mesh filename=robotiq_arg85_description/meshes/outer_finger_coarse.STL; visual mesh filename=robotiq_arg85_description/meshes/outer_finger_fine.STL
- added link left_outer_knuckle, mass 0.00684838849434396; collision mesh filename=robotiq_arg85_description/meshes/outer_knuckle_coarse.STL; visual mesh filename=robotiq_arg85_description/meshes/outer_knuckle_fine.STL
- added link right_inner_finger, mass 0.00724255346165744; collision mesh filename=robotiq_arg85_description/meshes/inner_finger_coarse.STL; visual mesh filename=robotiq_arg85_description/meshes/inner_finger_fine.STL
- added link right_inner_knuckle, mass 0.0110930853895903; collision mesh filename=robotiq_arg85_description/meshes/inner_knuckle_coarse.STL; visual mesh filename=robotiq_arg85_description/meshes/inner_knuckle_fine.STL
- added link right_outer_finger, mass 0.0273093985570947; collision mesh filename=robotiq_arg85_description/meshes/outer_finger_coarse.STL; visual mesh filename=robotiq_arg85_description/meshes/outer_finger_fine.STL
- added link right_outer_knuckle, mass 0.00684838849401352; collision mesh filename=robotiq_arg85_description/meshes/outer_knuckle_coarse.STL; visual mesh filename=robotiq_arg85_description/meshes/outer_knuckle_fine.STL
- added link robotiq_85_base_link, mass 0.30915; collision mesh filename=robotiq_arg85_description/meshes/robotiq_85_base_link_coars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; visual mesh filename=robotiq_arg85_description/meshes/robotiq_85_base_link_fine.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
Joints:
- added joint finger_joint: type revolute, parent robotiq_85_base_link, child left_outer_knuckle, origin xyz=0.0306011444260539 0 0.0627920162695395 rpy=0 0 0, axis 0 -1 0, limit lower=0 upper=0.725 effort=1000 velocity=2.0
- added joint left_inner_finger_joint: type revolute, parent left_inner_knuckle, child left_inner_finger, origin xyz=0.034585310861294 0 0.0454970193817975 rpy=0 0 0, axis 0 -1 0, limit lower=0 upper=0.8757 effort=1000 velocity=2.0, mimic joint=finger_joint multiplier=-1 offset=0
- added joint left_inner_knuckle_joint: type revolute, parent robotiq_85_base_link, child left_inner_knuckle, origin xyz=0.0127000000001501 0 0.0693074999999639 rpy=0 0 0, axis 0 -1 0, limit lower=0 upper=0.8757 effort=1000 velocity=2.0, mimic joint=finger_joint multiplier=1 offset=0
- added joint left_outer_finger_joint: type fixed, parent left_outer_knuckle, child left_outer_finger, origin xyz=0.0316910442266543 0 -0.00193396375724605 rpy=0 0 0, axis 0 -1 0
- added joint right_inner_finger_joint: type revolute, parent right_inner_knuckle, child right_inner_finger, origin xyz=0.0341060475457406 0 0.0458573878541688 rpy=0 0 0, axis 0 1 0, limit lower=0 upper=0.8757 effort=1000 velocity=2.0, mimic joint=finger_joint multiplier=1 offset=0
- added joint right_inner_knuckle_joint: type revolute, parent robotiq_85_base_link, child right_inner_knuckle, origin xyz=-0.0126999999998499 0 0.0693075000000361 rpy=0 0 3.14159265358979, axis 0 1 0, limit lower=0 upper=0.8757 effort=1000 velocity=2.0, mimic joint=finger_joint multiplier=-1 offset=0
- added joint right_outer_finger_joint: type fixed, parent right_outer_knuckle, child right_outer_finger, origin xyz=0.0317095909367246 0 -0.0016013564954687 rpy=0 0 0, axis 0 1 0
- added joint right_outer_knuckle_joint: type revolute, parent robotiq_85_base_link, child right_outer_knuckle, origin xyz=-0.0306011444258893 0 0.0627920162695395 rpy=0 0 3.14159265358979, axis 0 1 0, limit lower=0 upper=0.8757 effort=1000 velocity=2.0, mimic joint=finger_joint multiplier=-1 offset=0
- added joint test_name: type fixed, parent panda_link8, child robotiq_85_base_link, origin xyz=0 0 0 rpy=0 0 1.57

File: franka_description/robots/common/franka_robot.xacro (robot description, xacro)
@@ -5,7 +5,7 @@
     <xacro:include filename="$(find franka_description)/robots/common/franka_arm.xacro" />
     <xacro:franka_arm arm_id="${arm_id}" safety_distance="0.03" gazebo="${gazebo}" joint_limits="${joint_limits}"/>
-    <xacro:if value="${hand}">
-      <xacro:include filename="$(find franka_description)/robots/common/franka_hand.xacro"/>
-      <xacro:franka_hand
+    <!-- <xacro:if value="${hand}"> -->
+      <xacro:include filename="$(find robotiq_arg85_description)/robots/robotiq_arg85_description.urdf.xacro"/>
+      <xacro:robotiq_85
           arm_id="${arm_id}"
           rpy="0 0 ${-pi/4}"
@@ -14,7 +14,6 @@
           connected_to="${arm_id}_link8"
           safety_distance="0.03"
-          gazebo="${gazebo}"
        />
-    </xacro:if>
+    <!-- </xacro:if> -->
     <!-- Define additional Gazebo tags -->
     <xacro:if value="${gazebo}">
